Commit message: Added debugging and parameterized hardware

File: src/niryo_one_hardware/description/ros2_control/niryo_one.ros2_control.xacro (robot description, xacro)
@@ -1,63 +1,66 @@
 <?xml version="1.0"?>
 <robot xmlns:xacro="http://www.ros.org/wiki/xacro">
+	<xacro:arg name="params_path" default="$(find niryo_one_hardware)/config/niryo_one_hardware_params.yaml" />
+	<xacro:property name="params_path" value="$(arg params_path)" />
+	<xacro:property name="mp" value="${xacro.load_yaml(params_path)}" />
 	<xacro:macro name="niryo_one_ros2_control" params="name">
 		<ros2_control name="${name}" type="system">
 			<hardware>
 				<plugin>niryo_one_hardware/NiryoOneHardware</plugin>
-				<param name="hardware_version">2</param>  <!-- /niryo_one/hardware_version -->
-				<param name="use_sim">false</param>  <!-- ~fake_communication -->
+				<param name="hardware_version">${mp['hardware_version']}</param>  <!-- /niryo_one/hardware_version -->
+				<param name="use_sim">${mp['use_sim']}</param>  <!-- ~fake_communication -->
 				<!-- Fake Communication -->
-				<param name="stepper_1_home_position">0.0</param>  <!-- /niryo_one/motors/stepper_1_home_position -->
-				<param name="stepper_2_home_position">0.64</param>  <!-- /niryo_one/motors/stepper_2_home_position -->
-				<param name="stepper_3_home_position">-1.39</param>  <!-- /niryo_one/motors/stepper_3_home_position -->
-				<param name="stepper_4_home_position">0.0</param>  <!-- /niryo_one/motors/stepper_4_home_position -->
+				<param name="stepper_1_home_position">${mp['stepper_1_home_position']}</param>  <!-- /niryo_one/motors/stepper_1_home_position -->
+				<param name="stepper_2_home_position">${mp['stepper_2_home_position']}</param>  <!-- /niryo_one/motors/stepper_2_home_position -->
+				<param name="stepper_3_home_position">${mp['stepper_3_home_position']}</param>  <!-- /niryo_one/motors/stepper_3_home_position -->
+				<param name="stepper_4_home_position">${mp['stepper_4_home_position']}</param>  <!-- /niryo_one/motors/stepper_4_home_position -->
 				<!-- Niryo One Communication -->
-				<param name="can_enabled">true</param>  <!-- ~can_enabled -->
-				<param name="dxl_enabled">true</param>  <!-- ~dxl_enabled -->
-				<param name="niryo_one_hw_check_connection_frequency">2.0</param>  <!-- niryo_one_hw_check_connection_frequency -->
-				<param name="reboot">true</param>  <!-- /niryo_one/reboot_when_auto_change_version -->
+				<param name="can_enabled">${mp['can_enabled']}</param>  <!-- ~can_enabled -->
+				<param name="dxl_enabled">${mp['dxl_enabled']}</param>  <!-- ~dxl_enabled -->
+				<param name="niryo_one_hw_check_connection_frequency">${mp['niryo_one_hw_check_connection_frequency']}</param>  <!-- niryo_one_hw_check_connection_frequency -->
+				<param name="reboot">${mp['reboot']}</param>  <!-- /niryo_one/reboot_when_auto_change_version -->
 				<!-- Can Communication -->
-				<param name="spi_channel">0</param>  <!-- ~spi_channel -->
-				<param name="spi_baudrate">1000000</param>  <!-- ~spi_baudrate -->
-				<param name="gpio_can_interrupt">25</param>  <!-- ~gpio_can_interrupt -->
-				<param name="can_hw_control_loop_frequency">1500.0</param>  <!-- ~can_hardware_control_loop_frequency -->
-				<param name="can_hw_write_frequency">50.0</param>  <!-- ~can_hardware_write_frequency -->
-				<param name="can_hw_check_connection_frequency">3.0</param>  <!-- ~can_hardware_check_connection_frequency -->
-				<param name="calibration_timeout">40</param>  <!-- ~calibration_timeout -->
-				<param name="required_steppers_ids">1,2,3</param>  <!-- /niryo_one/motors/can_required_motors -->
-				<param name="allowed_steppers_ids">1,2,3,6,7</param>  <!-- /niryo_one/motors/can_authorized_motors -->
-				<param name="gear_ratio_1">6.0625</param>  <!-- /niryo_one/motors/stepper_1_gear_ratio -->
-				<param name="gear_ratio_2">8.3125</param>  <!-- /niryo_one/motors/stepper_2_gear_ratio -->
-				<param name="gear_ratio_3">7.875</param>  <!-- /niryo_one/motors/stepper_3_gear_ratio -->
-				<param name="gear_ratio_4">5.0</param>  <!-- /niryo_one/motors/stepper_4_gear_ratio -->
-				<param name="gear_ratio_6">5.0</param>  <!-- /niryo_one/motors/stepper_6_gear_ratio -->
-				<param name="gear_ratio_7">5.0</param>  <!-- /niryo_one/motors/stepper_7_gear_ratio -->
-				<param name="home_position_1">0.0</param>  <!-- /niryo_one/motors/stepper_1_home_position -->
-				<param name="home_position_2">0.640187</param>  <!-- /niryo_one/motors/stepper_2_home_position -->
-				<param name="home_position_3">-1.397485</param>  <!-- /niryo_one/motors/stepper_3_home_position -->
-				<param name="home_position_4">0.0</param>  <!-- /niryo_one/motors/stepper_4_home_position -->
-				<param name="offset_position_1">3.05433</param>  <!-- /niryo_one/motors/stepper_1_offset_position -->
-				<param name="offset_position_2">0.640187</param>  <!-- /niryo_one/motors/stepper_2_offset_position -->
-				<param name="offset_position_3">-1.397485</param>  <!-- /niryo_one/motors/stepper_3_offset_position -->
-				<param name="offset_position_4">2.791</param>  <!-- /niryo_one/motors/stepper_4_offset_position -->
-				<param name="direction_1">-1.0</param>  <!-- /niryo_one/motors/stepper_1_direction -->
-				<param name="direction_2">-1.0</param>  <!-- /niryo_one/motors/stepper_2_direction -->
-				<param name="direction_3">1.0</param>  <!-- /niryo_one/motors/stepper_3_direction -->
-				<param name="direction_4">-1.0</param>  <!-- /niryo_one/motors/stepper_4_direction -->
-				<param name="max_effort_1">90</param>  <!-- /niryo_one/motors/stepper_1_max_effort -->
-				<param name="max_effort_2">130</param>  <!-- /niryo_one/motors/stepper_2_max_effort -->
-				<param name="max_effort_3">120</param>  <!-- /niryo_one/motors/stepper_3_max_effort -->
-				<param name="max_effort_4">90</param>  <!-- /niryo_one/motors/stepper_4_max_effort -->
-				<param name="max_effort_6">90</param>  <!-- /niryo_one/motors/stepper_6_max_effort -->
-				<param name="max_effort_7">90</param>  <!-- /niryo_one/motors/stepper_7_max_effort -->
+				<param name="spi_channel">${mp['spi_channel']}</param>  <!-- ~spi_channel -->
+				<param name="spi_baudrate">${mp['spi_baudrate']}</param>  <!-- ~spi_baudrate -->
+				<param name="gpio_can_interrupt">${mp['gpio_can_interrupt']}</param>  <!-- ~gpio_can_interrupt -->
+				<param name="can_hw_control_loop_frequency">${mp['can_hw_control_loop_frequency']}</param>  <!-- ~can_hardware_control_loop_frequency -->
+				<param name="can_hw_write_frequency">${mp['can_hw_write_frequency']}</param>  <!-- ~can_hardware_write_frequency -->
+				<param name="can_hw_check_connection_frequency">${mp['can_hw_check_connection_frequency']}</param>  <!-- ~can_hardware_check_connection_frequency -->
+				<param name="calibration_timeout">${mp['calibration_timeout']}</param>  <!-- ~calibration_timeout -->
+				<param name="required_steppers_ids">${mp['required_steppers_ids']}</param>  <!-- /niryo_one/motors/can_required_motors -->
+				<param name="allowed_steppers_ids">${mp['allowed_steppers_ids']}</param>  <!-- /niryo_one/motors/can_authorized_motors -->
+				<param name="gear_ratio_1">${mp['gear_ratio_1']}</param>  <!-- /niryo_one/motors/stepper_1_gear_ratio -->
+				<param name="gear_ratio_2">${mp['gear_ratio_2']}</param>  <!-- /niryo_one/motors/stepper_2_gear_ratio -->
+				<param name="gear_ratio_3">${mp['gear_ratio_3']}</param>  <!-- /niryo_one/motors/stepper_3_gear_ratio -->
+				<param name="gear_ratio_4">${mp['gear_ratio_4']}</param>  <!-- /niryo_one/motors/stepper_4_gear_ratio -->
+				<param name="gear_ratio_6">${mp['gear_ratio_6']}</param>  <!-- /niryo_one/motors/stepper_6_gear_ratio -->
+				<param name="gear_ratio_7">${mp['gear_ratio_7']}</param>  <!-- /niryo_one/motors/stepper_7_gear_ratio -->
+				<param name="home_position_1">${mp['home_position_1']}</param>  <!-- /niryo_one/motors/stepper_1_home_position -->
+				<param name="home_position_2">${mp['home_position_2']}</param>  <!-- /niryo_one/motors/stepper_2_home_position -->
+				<param name="home_position_3">${mp['home_position_3']}</param>  <!-- /niryo_one/motors/stepper_3_home_position -->
+				<param name="home_position_4">${mp['home_position_4']}</param>  <!-- /niryo_one/motors/stepper_4_home_position -->
+				<param name="offset_position_1">${mp['offset_position_1']}</param>  <!-- /niryo_one/motors/stepper_1_offset_position -->
+				<param name="offset_position_2">${mp['offset_position_2']}</param>  <!-- /niryo_one/motors/stepper_2_offset_position -->
+				<param name="offset_position_3">${mp['offset_position_3']}</param>  <!-- /niryo_one/motors/stepper_3_offset_position -->
+				<param name="offset_position_4">${mp['offset_position_4']}</param>  <!-- /niryo_one/motors/stepper_4_offset_position -->
+				<param name="direction_1">${mp['direction_1']}</param>  <!-- /niryo_one/motors/stepper_1_direction -->
+				<param name="direction_2">${mp['direction_2']}</param>  <!-- /niryo_one/motors/stepper_2_direction -->
+				<param name="direction_3">${mp['direction_3']}</param>  <!-- /niryo_one/motors/stepper_3_direction -->
+				<param name="direction_4">${mp['direction_4']}</param>  <!-- /niryo_one/motors/stepper_4_direction -->
+				<param name="max_effort_1">${mp['max_effort_1']}</param>  <!-- /niryo_one/motors/stepper_1_max_effort -->
+				<param name="max_effort_2">${mp['max_effort_2']}</param>  <!-- /niryo_one/motors/stepper_2_max_effort -->
+				<param name="max_effort_3">${mp['max_effort_3']}</param>  <!-- /niryo_one/motors/stepper_3_max_effort -->
+				<param name="max_effort_4">${mp['max_effort_4']}</param>  <!-- /niryo_one/motors/stepper_4_max_effort -->
+				<param name="max_effort_6">${mp['max_effort_6']}</param>  <!-- /niryo_one/motors/stepper_6_max_effort -->
+				<param name="max_effort_7">${mp['max_effort_7']}</param>  <!-- /niryo_one/motors/stepper_7_max_effort -->
 				<!-- Dxl Communication -->
-				<param name="device_name">/dev/ttyAMA0</param>  <!-- ~dxl_uart_device_name -->
-				<param name="uart_baudrate">1000000</param>  <!-- ~dxl_baudrate -->
-				<param name="dxl_hw_control_loop_frequency">100.0</param>  <!-- ~dxl_hardware_control_loop_frequency -->
-				<param name="dxl_hw_write_frequency">50.0</param>  <!-- ~dxl_hw_write_frequency -->
-				<param name="dxl_hw_data_read_frequency">15.0</param>  <!-- ~dxl_hw_data_read_frequency -->
-				<param name="dxl_hw_status_read_frequency">0.5</param>  <!-- ~dxl_hw_status_read_frequency -->
-				<param name="required_dxl_ids">2,3,6</param>  <!-- /niryo_one/motors/dxl_required_motors -->
-				<param name="allowed_dxl_ids">2,3,6,11,12,13,31</param>  <!-- /niryo_one/motors/dxl_authorized_motors -->
+				<param name="device_name">${mp['device_name']}</param>  <!-- ~dxl_uart_device_name -->
+				<param name="uart_baudrate">${mp['uart_baudrate']}</param>  <!-- ~dxl_baudrate -->
+				<param name="dxl_hw_control_loop_frequency">${mp['dxl_hw_control_loop_frequency']}</param>  <!-- ~dxl_hardware_control_loop_frequency -->
+				<param name="dxl_hw_write_frequency">${mp['dxl_hw_write_frequency']}</param>  <!-- ~dxl_hw_write_frequency -->
+				<param name="dxl_hw_data_read_frequency">${mp['dxl_hw_data_read_frequency']}</param>  <!-- ~dxl_hw_data_read_frequency -->
+				<param name="dxl_hw_status_read_frequency">${mp['dxl_hw_status_read_frequency']}</param>  <!-- ~dxl_hw_status_read_frequency -->
+				<param name="required_dxl_ids">${mp['required_dxl_ids']}</param>  <!-- /niryo_one/motors/dxl_required_motors -->
+				<param name="allowed_dxl_ids">${mp['allowed_dxl_ids']}</param>  <!-- /niryo_one/motors/dxl_authorized_motors -->
 			</hardware>
 			<joint name="joint_1">

Commit message: Current attempt at getting stuff working

File: src/niryo_one_hardware/description/ros2_control/niryo_one.ros2_control.xacro (robot description, xacro)
@@ -5,7 +5,7 @@
 	<xacro:property name="mp" value="${xacro.load_yaml(params_path)}" />
 	<xacro:macro name="niryo_one_ros2_control" params="name">
-		<ros2_control name="${name}" type="system">
+		<ros2_control name="${name}_can" type="system">
 			<hardware>
-				<plugin>niryo_one_hardware/NiryoOneHardware</plugin>
+				<plugin>niryo_one_hardware/NiryoOneHardwareCan</plugin>
 				<param name="hardware_version">${mp['hardware_version']}</param>  <!-- /niryo_one/hardware_version -->
 				<param name="use_sim">${mp['use_sim']}</param>  <!-- ~fake_communication -->
@@ -54,15 +54,14 @@
 				<param name="max_effort_6">${mp['max_effort_6']}</param>  <!-- /niryo_one/motors/stepper_6_max_effort -->
 				<param name="max_effort_7">${mp['max_effort_7']}</param>  <!-- /niryo_one/motors/stepper_7_max_effort -->
-				<!-- Dxl Communication -->
-				<param name="device_name">${mp['device_name']}</param>  <!-- ~dxl_uart_device_name -->
-				<param name="uart_baudrate">${mp['uart_baudrate']}</param>  <!-- ~dxl_baudrate -->
-				<param name="dxl_hw_control_loop_frequency">${mp['dxl_hw_control_loop_frequency']}</param>  <!-- ~dxl_hardware_control_loop_frequency -->
-				<param name="dxl_hw_write_frequency">${mp['dxl_hw_write_frequency']}</param>  <!-- ~dxl_hw_write_frequency -->
-				<param name="dxl_hw_data_read_frequency">${mp['dxl_hw_data_read_frequency']}</param>  <!-- ~dxl_hw_data_read_frequency -->
-				<param name="dxl_hw_status_read_frequency">${mp['dxl_hw_status_read_frequency']}</param>  <!-- ~dxl_hw_status_read_frequency -->
-				<param name="required_dxl_ids">${mp['required_dxl_ids']}</param>  <!-- /niryo_one/motors/dxl_required_motors -->
-				<param name="allowed_dxl_ids">${mp['allowed_dxl_ids']}</param>  <!-- /niryo_one/motors/dxl_authorized_motors -->
 			</hardware>
 			<joint name="joint_1">
+				<param name="id">1</param>
+				<param name="name">Stepper Axis 1</param>
+				<param name="gear_ratio">${mp['gear_ratio_1']}</param>
+				<param name="home_position">${mp['home_position_1']}</param>
+				<param name="offset_position">${mp['offset_position_1']}</param>
+				<param name="direction">${mp['direction_1']}</param>
+				<param name="max_effort">${mp['max_effort_1']}</param>
+				<param name="firmware_version">2.0.0</param>
 				<command_interface name="position">
 					<param name="min">${-2*pi}</param>
@@ -73,10 +72,27 @@
 					<param name="max">3.15</param>
 				</command_interface>
+				<command_interface name="torque" />
+				<command_interface name="mirco_steps" />
+				<command_interface name="max_effort" />
 				<state_interface name="position">
 					<param name="initial_value">0.0</param>
 				</state_interface>
 				<state_interface name="velocity" />
+				<state_interface name="torque" />
+				<state_interface name="temperature" />
+				<state_interface name="hardware_error" />
+				<state_interface name="enabled">
+					<param name="initial_value">false</param>
+				</state_interface>
 			</joint>
 			<joint name="joint_2">
+				<param name="id">2</param>
+				<param name="name">Stepper Axis 2</param>
+				<param name="gear_ratio">${mp['gear_ratio_2']}</param>
+				<param name="home_position">${mp['home_position_2']}</param>
+				<param name="offset_position">${mp['offset_position_2']}</param>
+				<param name="direction">${mp['direction_2']}</param>
+				<param name="max_effort">${mp['max_effort_2']}</param>
+				<param name="firmware_version">2.0.0</param>
 				<command_interface name="position">
 					<param name="min">${-2*pi}</param>
@@ -87,10 +103,27 @@
 					<param name="max">3.15</param>
 				</command_interface>
+				<command_interface name="torque" />
+				<command_interface name="mirco_steps" />
+				<command_interface name="max_effort" />
 				<state_interface name="position">
 					<param name="initial_value">0.64</param>
 				</state_interface>
 				<state_interface name="velocity" />
+				<state_interface name="torque" />
+				<state_interface name="temperature" />
+				<state_interface name="hardware_error" />
+				<state_interface name="enabled">
+					<param name="initial_value">false</param>
+				</state_interface>
 			</joint>
 			<joint name="joint_3">
+				<param name="id">3</param>
+				<param name="name">Stepper Axis 3</param>
+				<param name="gear_ratio">${mp['gear_ratio_3']}</param>
+				<param name="home_position">${mp['home_position_3']}</param>
+				<param name="offset_position">${mp['offset_position_3']}</param>
+				<param name="direction">${mp['direction_3']}</param>
+				<param name="max_effort">${mp['max_effort_3']}</param>
+				<param name="firmware_version">2.0.0</param>
 				<command_interface name="position">
 					<param name="min">${-pi}</param>
@@ -101,69 +134,18 @@
 					<param name="max">3.15</param>
 				</command_interface>
+				<command_interface name="torque" />
+				<command_interface name="mirco_steps" />
+				<command_interface name="max_effort" />
 				<state_interface name="position">
 					<param name="initial_value">-1.39</param>
 				</state_interface>
 				<state_interface name="velocity" />
+				<state_interface name="torque" />
+				<state_interface name="temperature" />
+				<state_interface name="hardware_error" />
+				<state_interface name="enabled">
+					<param name="initial_value">false</param>
+				</state_interface>
 			</joint>
-			<joint name="joint_4">
-				<command_interface name="position">
-					<param name="min">${-2*pi}</param>
-					<param name="max">${2*pi}</param>
-				</command_interface>
-				<command_interface name="velocity">
-					<param name="min">-3.2</param>
-					<param name="max">3.2</param>
-				</command_interface>
-				<state_interface name="position">
-					<param name="initial_value">0.0</param>
-				</state_interface>
-				<state_interface name="velocity" />
-			</joint>
-			<joint name="joint_5">
-				<command_interface name="position">
-					<param name="min">${-2*pi}</param>
-					<param name="max">${2*pi}</param>
-				</command_interface>
-				<command_interface name="velocity">
-					<param name="min">-3.2</param>
-					<param name="max">3.2</param>
-				</command_interface>
-				<state_interface name="position">
-					<param name="initial_value">0.0</param>
-				</state_interface>
-				<state_interface name="velocity" />
-			</joint>
-			<joint name="joint_6">
-				<command_interface name="position">
-					<param name="min">${-2*pi}</param>
-					<param name="max">${2*pi}</param>
-				</command_interface>
-				<command_interface name="velocity">
-					<param name="min">-3.2</param>
-					<param name="max">3.2</param>
-				</command_interface>
-				<state_interface name="position">
-					<param name="initial_value">0.0</param>
-				</state_interface>
-				<state_interface name="velocity" />
-			</joint>
-			<gpio name="hardware">
-				<command_interface name="test_motors" />
-				<command_interface name="calibrate_motors" />
-				<command_interface name="request_new_calibration" />
-				<command_interface name="activate_learning_mode" />
-				<command_interface name="activate_leds" />
-				<command_interface name="ping_and_set_dxl_tool" />
-				<command_interface name="ping_and_set_conveyor" />
-				<command_interface name="control_conveyor" />
-				<command_interface name="update_id_conveyor" />
-				<command_interface name="open_gripper" />
-				<command_interface name="close_gripper" />
-				<command_interface name="pull_air_vacuum_pump" />
-				<command_interface name="push_air_vacuum_pump" />
-				<command_interface name="change_hardware_version" />
-				<command_interface name="send_custom_dxl_value" />
-				<command_interface name="reboot_motors" />
-			</gpio>
 		</ros2_control>
 	</xacro:macro>
