Commit message: Add niryo_one_hardware from niryo_one_hardware branch

File: src/niryo_one_hardware/description/ros2_control/niryo_one.ros2_control.xacro (robot description, xacro)
@@ -4,16 +4,4 @@
 	<xacro:property name="params_path" value="$(arg params_path)" />
 	<xacro:property name="mp" value="${xacro.load_yaml(params_path)}" />
-	<xacro:property name="motor_type_xl320" value="1" />
-	<xacro:property name="motor_type_xl430" value="2" />
-	<xacro:property name="xl320_total_angle" value="296.67" />
-	<xacro:property name="xl320_max_position" value="1022" />
-	<xacro:property name="xl320_min_position" value="0" />
-	<xacro:property name="xl320_middle_position" value="511" />
-	<xacro:property name="xl320_total_range_position" value="1023" />
-	<xacro:property name="xl430_total_angle" value="360.36" />
-	<xacro:property name="xl430_max_position" value="4094" />
-	<xacro:property name="xl430_min_position" value="0" />
-	<xacro:property name="xl430_middle_position" value="2047" />
-	<xacro:property name="xl430_total_range_position" value="4095" />
 	<xacro:macro name="niryo_one_ros2_control" params="name">
 		<ros2_control name="${name}_can" type="system">
@@ -86,5 +74,7 @@
 				<command_interface name="torque" />
 				<command_interface name="mirco_steps" />
-				<command_interface name="max_effort" />
+				<command_interface name="max_effort">
+					<param name="max">1</param>
+				</command_interface>
 				<state_interface name="position">
 					<param name="initial_value">${mp['home_position_1']}</param>
@@ -128,5 +118,7 @@
 				<command_interface name="torque" />
 				<command_interface name="mirco_steps" />
-				<command_interface name="max_effort" />
+				<command_interface name="max_effort">
+					<param name="max">1</param>
+				</command_interface>
 				<state_interface name="position">
 					<param name="initial_value">${mp['home_position_2']}</param>
@@ -170,5 +162,7 @@
 				<command_interface name="torque" />
 				<command_interface name="mirco_steps" />
-				<command_interface name="max_effort" />
+				<command_interface name="max_effort">
+					<param name="max">1</param>
+				</command_interface>
 				<state_interface name="position">
 					<param name="initial_value">${mp['home_position_3']}</param>
@@ -211,11 +205,9 @@
 				<param name="dxl_hw_data_read_frequency">${mp['dxl_hw_data_read_frequency']}</param>
 				<param name="dxl_hw_status_read_frequency">${mp['dxl_hw_status_read_frequency']}</param>
-				<param name="allowed_dxl_ids">${mp['allowed_dxl_ids']}</param>
 			</hardware>
 			<joint name="joint_4">
 				<param name="id">2</param>
 				<param name="name">Servo Axis 4</param>
-				<param name="type">${motor_type_xl430}</param>
-				<param name="home_position">${xl430_middle_position}</param>
+				<param name="type">2</param>  <!-- XL430 -->
 				<command_interface name="position">
 					<param name="min">${limit_low_forearm_rotation}</param>
@@ -229,5 +221,5 @@
 				<command_interface name="led" />
 				<state_interface name="position">
-					<param name="initial_value">${xl430_middle_position}</param>
+					<param name="initial_value">2047</param>
 				</state_interface>
 				<state_interface name="velocity" />
@@ -241,6 +233,5 @@
 				<param name="id">3</param>
 				<param name="name">Servo Axis 5</param>
-				<param name="type">${motor_type_xl430}</param>
-				<param name="home_position">${xl430_middle_position}</param>
+				<param name="type">2</param>  <!-- XL430 -->
 				<command_interface name="position">
 					<param name="min">${limit_low_wrist_rotation}</param>
@@ -254,5 +245,5 @@
 				<command_interface name="led" />
 				<state_interface name="position">
-					<param name="initial_value">${xl430_middle_position}</param>
+					<param name="initial_value">2047</param>
 				</state_interface>
 				<state_interface name="velocity" />
@@ -266,6 +257,5 @@
 				<param name="id">6</param>
 				<param name="name">Servo Axis 6</param>
-				<param name="type">${motor_type_xl320}</param>
-				<param name="home_position">${xl320_middle_position}</param>
+				<param name="type">1</param>  <!-- XL320 -->
 				<command_interface name="position">
 					<param name="min">${limit_low_hand_rotation}</param>
@@ -304,5 +294,5 @@
 				<command_interface name="led" />
 				<state_interface name="position">
-					<param name="initial_value">${xl320_middle_position}</param>
+					<param name="initial_value">511</param>
 				</state_interface>
 				<state_interface name="velocity" />

Commit message: Coded DXL motor controller

File: src/niryo_one_hardware/description/ros2_control/niryo_one.ros2_control.xacro (robot description, xacro)
@@ -4,4 +4,16 @@
 	<xacro:property name="params_path" value="$(arg params_path)" />
 	<xacro:property name="mp" value="${xacro.load_yaml(params_path)}" />
+	<xacro:property name="motor_type_xl320" value="1" />
+	<xacro:property name="motor_type_xl430" value="2" />
+	<xacro:property name="xl320_total_angle" value="296.67" />
+	<xacro:property name="xl320_max_position" value="1022" />
+	<xacro:property name="xl320_min_position" value="0" />
+	<xacro:property name="xl320_middle_position" value="511" />
+	<xacro:property name="xl320_total_range_position" value="1023" />
+	<xacro:property name="xl430_total_angle" value="360.36" />
+	<xacro:property name="xl430_max_position" value="4094" />
+	<xacro:property name="xl430_min_position" value="0" />
+	<xacro:property name="xl430_middle_position" value="2047" />
+	<xacro:property name="xl430_total_range_position" value="4095" />
 	<xacro:macro name="niryo_one_ros2_control" params="name">
 		<ros2_control name="${name}_can" type="system">
@@ -73,7 +85,5 @@
 				<command_interface name="torque" />
 				<command_interface name="mirco_steps" />
-				<command_interface name="max_effort">
-					<param name="max">1</param>
-				</command_interface>
+				<command_interface name="max_effort" />
 				<state_interface name="position">
 					<param name="initial_value">${mp['home_position_1']}</param>
@@ -116,7 +126,5 @@
 				<command_interface name="torque" />
 				<command_interface name="mirco_steps" />
-				<command_interface name="max_effort">
-					<param name="max">1</param>
-				</command_interface>
+				<command_interface name="max_effort" />
 				<state_interface name="position">
 					<param name="initial_value">${mp['home_position_2']}</param>
@@ -159,7 +167,5 @@
 				<command_interface name="torque" />
 				<command_interface name="mirco_steps" />
-				<command_interface name="max_effort">
-					<param name="max">1</param>
-				</command_interface>
+				<command_interface name="max_effort" />
 				<state_interface name="position">
 					<param name="initial_value">${mp['home_position_3']}</param>
@@ -206,5 +212,6 @@
 				<param name="id">2</param>
 				<param name="name">Servo Axis 4</param>
-				<param name="type">2</param>  <!-- XL430 -->
+				<param name="type">${motor_type_xl430}</param>
+				<param name="home_position">${xl430_middle_position}</param>
 				<command_interface name="position">
 					<param name="min">${limit_low_forearm_rotation}</param>
@@ -217,5 +224,5 @@
 				<command_interface name="led" />
 				<state_interface name="position">
-					<param name="initial_value">2047</param>
+					<param name="initial_value">${xl430_middle_position}</param>
 				</state_interface>
 				<state_interface name="velocity" />
@@ -229,5 +236,6 @@
 				<param name="id">3</param>
 				<param name="name">Servo Axis 5</param>
-				<param name="type">2</param>  <!-- XL430 -->
+				<param name="type">${motor_type_xl430}</param>
+				<param name="home_position">${xl430_middle_position}</param>
 				<command_interface name="position">
 					<param name="min">${limit_low_wrist_rotation}</param>
@@ -240,5 +248,5 @@
 				<command_interface name="led" />
 				<state_interface name="position">
-					<param name="initial_value">2047</param>
+					<param name="initial_value">${xl430_middle_position}</param>
 				</state_interface>
 				<state_interface name="velocity" />
@@ -252,5 +260,6 @@
 				<param name="id">6</param>
 				<param name="name">Servo Axis 6</param>
-				<param name="type">1</param>  <!-- XL320 -->
+				<param name="type">${motor_type_xl320}</param>
+				<param name="home_position">${xl320_middle_position}</param>
 				<command_interface name="position">
 					<param name="min">${limit_low_hand_rotation}</param>
@@ -263,5 +272,5 @@
 				<command_interface name="led" />
 				<state_interface name="position">
-					<param name="initial_value">511</param>
+					<param name="initial_value">${xl320_middle_position}</param>
 				</state_interface>
 				<state_interface name="velocity" />
