Commit message: Woring on adding the ros interface stuff to the controller

File: src/niryo_one_description/urdf/v2/niryo_one_description.urdf.xacro (robot description, xacro)
@@ -29,4 +29,5 @@
 		<xacro:property name="limit_up_hand_rotation" value="2.57436" />
 		<!-- Links -->
+		<link name="world" />
 		<xacro:create_link
 			link_name="base_link"

File: src/niryo_one_hardware/description/ros2_control/niryo_one.ros2_control.xacro (robot description, xacro)
@@ -148,4 +148,22 @@
 				<state_interface name="velocity" />
 			</joint>
+			<gpio name="hardware">
+				<command_interface name="test_motors" />
+				<command_interface name="calibrate_motors" />
+				<command_interface name="request_new_calibration" />
+				<command_interface name="activate_learning_mode" />
+				<command_interface name="activate_leds" />
+				<command_interface name="ping_and_set_dxl_tool" />
+				<command_interface name="ping_and_set_conveyor" />
+				<command_interface name="control_conveyor" />
+				<command_interface name="update_id_conveyor" />
+				<command_interface name="open_gripper" />
+				<command_interface name="close_gripper" />
+				<command_interface name="pull_air_vacuum_pump" />
+				<command_interface name="push_air_vacuum_pump" />
+				<command_interface name="change_hardware_version" />
+				<command_interface name="send_custom_dxl_value" />
+				<command_interface name="reboot_motors" />
+			</gpio>
 		</ros2_control>
 	</xacro:macro>

File: src/niryo_one_hardware/description/urdf/niryo_one.urdf.xacro (robot description, xacro)
@@ -4,6 +4,4 @@
 	<!-- <xacro:include filename="$(find niryo_one_description)/urdf/v2/niryo_one.urdf.xacro" /> -->
 	<xacro:include filename="$(find niryo_one_description)/urdf/v2/niryo_one_description.urdf.xacro" />
-	<!-- create link fixed to the "world" -->
-	<link name="world" />
 	<xacro:niryo_one_description />
 	<!-- Import niryo_one_ros2_control description -->

Commit message: Got CAN motors working and started work on DXL motors

File: src/niryo_one_description/urdf/v2/niryo_one_description.urdf.xacro (robot description, xacro)
@@ -4,28 +4,4 @@
 		<!-- Helper macro-->
 		<xacro:include filename="$(find niryo_one_description)/urdf/v2/inc/create_link.xacro" />
-		<!-- Properties -->
-		<xacro:property name="distance_origin_shoulder_z" value="0.103" />
-		<xacro:property name="distance_shoulder_arm_z" value="0.080" />
-		<xacro:property name="distance_arm_elbow_x" value="0.210" />
-		<xacro:property name="distance_arm_elbow_y" value="0.0" />
-		<xacro:property name="distance_elbow_forearm_x" value="0.0415" />
-		<xacro:property name="distance_elbow_forearm_y" value="0.030" />
-		<xacro:property name="distance_forearm_wrist_z" value="0.180" />
-		<xacro:property name="distance_wrist_hand_x" value="0.0164" />
-		<xacro:property name="distance_wrist_hand_y" value="-0.0055" />
-		<xacro:property name="distance_hand_tool" value="0.0073" />
-		<xacro:property name="PI" value="3.14159265359" />
-		<xacro:property name="limit_low_shoulder_rotation" value="-3.05433" />
-		<xacro:property name="limit_up_shoulder_rotation" value="3.05433" />
-		<xacro:property name="limit_low_arm_rotation" value="-1.57080" />
-		<xacro:property name="limit_up_arm_rotation" value="0.640187" />
-		<xacro:property name="limit_low_elbow_rotation" value="-1.397485" />
-		<xacro:property name="limit_up_elbow_rotation" value="${PI/2}" />
-		<xacro:property name="limit_low_forearm_rotation" value="-3.05433" />
-		<xacro:property name="limit_up_forearm_rotation" value="3.05433" />
-		<xacro:property name="limit_low_wrist_rotation" value="-1.74533" />
-		<xacro:property name="limit_up_wrist_rotation" value="1.91986" />
-		<xacro:property name="limit_low_hand_rotation" value="-2.57436" />
-		<xacro:property name="limit_up_hand_rotation" value="2.57436" />
 		<!-- Links -->
 		<link name="world" />

File: src/niryo_one_hardware/description/ros2_control/niryo_one.ros2_control.xacro (robot description, xacro)
@@ -65,16 +65,17 @@
 				<param name="firmware_version">2.0.0</param>
 				<command_interface name="position">
-					<param name="min">${-2*pi}</param>
-					<param name="max">${2*pi}</param>
-				</command_interface>
-				<command_interface name="velocity">
-					<param name="min">-3.15</param>
-					<param name="max">3.15</param>
+					<param name="min">${limit_low_shoulder_rotation}</param>
+					<param name="max">${limit_up_shoulder_rotation}</param>
+				</command_interface>
+				<command_interface name="velocity">
+					<param name="max">1.0</param>
 				</command_interface>
 				<command_interface name="torque" />
 				<command_interface name="mirco_steps" />
-				<command_interface name="max_effort" />
-				<state_interface name="position">
-					<param name="initial_value">0.0</param>
+				<command_interface name="max_effort">
+					<param name="max">1</param>
+				</command_interface>
+				<state_interface name="position">
+					<param name="initial_value">${mp['home_position_1']}</param>
 				</state_interface>
 				<state_interface name="velocity" />
@@ -83,5 +84,16 @@
 				<state_interface name="hardware_error" />
 				<state_interface name="enabled">
-					<param name="initial_value">false</param>
+					<param name="initial_value">true</param>
+				</state_interface>
+				<state_interface name="hw_fail_counter" />
+				<state_interface name="last_time_read" />
+				<state_interface name="firmware_version_major">
+					<param name="initial_value">2</param>
+				</state_interface>
+				<state_interface name="firmware_version_minor">
+					<param name="initial_value">0</param>
+				</state_interface>
+				<state_interface name="firmware_version_patch">
+					<param name="initial_value">0</param>
 				</state_interface>
 			</joint>
@@ -96,16 +108,17 @@
 				<param name="firmware_version">2.0.0</param>
 				<command_interface name="position">
-					<param name="min">${-2*pi}</param>
-					<param name="max">${2*pi}</param>
-				</command_interface>
-				<command_interface name="velocity">
-					<param name="min">-3.15</param>
-					<param name="max">3.15</param>
+					<param name="min">${limit_low_arm_rotation}</param>
+					<param name="max">${limit_up_arm_rotation}</param>
+				</command_interface>
+				<command_interface name="velocity">
+					<param name="max">1.0</param>
 				</command_interface>
 				<command_interface name="torque" />
 				<command_interface name="mirco_steps" />
-				<command_interface name="max_effort" />
-				<state_interface name="position">
-					<param name="initial_value">0.64</param>
+				<command_interface name="max_effort">
+					<param name="max">1</param>
+				</command_interface>
+				<state_interface name="position">
+					<param name="initial_value">${mp['home_position_2']}</param>
 				</state_interface>
 				<state_interface name="velocity" />
@@ -114,5 +127,16 @@
 				<state_interface name="hardware_error" />
 				<state_interface name="enabled">
-					<param name="initial_value">false</param>
+					<param name="initial_value">true</param>
+				</state_interface>
+				<state_interface name="hw_fail_counter" />
+				<state_interface name="last_time_read" />
+				<state_interface name="firmware_version_major">
+					<param name="initial_value">2</param>
+				</state_interface>
+				<state_interface name="firmware_version_minor">
+					<param name="initial_value">0</param>
+				</state_interface>
+				<state_interface name="firmware_version_patch">
+					<param name="initial_value">0</param>
 				</state_interface>
 			</joint>
@@ -127,16 +151,17 @@
 				<param name="firmware_version">2.0.0</param>
 				<command_interface name="position">
-					<param name="min">${-pi}</param>
-					<param name="max">${pi}</param>
-				</command_interface>
-				<command_interface name="velocity">
-					<param name="min">-3.15</param>
-					<param name="max">3.15</param>
+					<param name="min">${limit_low_elbow_rotation}</param>
+					<param name="max">${limit_up_elbow_rotation}</param>
+				</command_interface>
+				<command_interface name="velocity">
+					<param name="max">1.0</param>
 				</command_interface>
 				<command_interface name="torque" />
 				<command_interface name="mirco_steps" />
-				<command_interface name="max_effort" />
-				<state_interface name="position">
-					<param name="initial_value">-1.39</param>
+				<command_interface name="max_effort">
+					<param name="max">1</param>
+				</command_interface>
+				<state_interface name="position">
+					<param name="initial_value">${mp['home_position_3']}</param>
 				</state_interface>
 				<state_interface name="velocity" />
@@ -145,6 +170,105 @@
 				<state_interface name="hardware_error" />
 				<state_interface name="enabled">
-					<param name="initial_value">false</param>
-				</state_interface>
+					<param name="initial_value">true</param>
+				</state_interface>
+				<state_interface name="hw_fail_counter" />
+				<state_interface name="last_time_read" />
+				<state_interface name="firmware_version_major">
+					<param name="initial_value">2</param>
+				</state_interface>
+				<state_interface name="firmware_version_minor">
+					<param name="initial_value">0</param>
+				</state_interface>
+				<state_interface name="firmware_version_patch">
+					<param name="initial_value">0</param>
+				</state_interface>
+			</joint>
+		</ros2_control>
+		<ros2_control name="${name}_dxl" type="system">
+			<hardware>
+				<plugin>niryo_one_hardware/NiryoOneHardwareDxl</plugin>
+				<param name="hardware_version">${mp['hardware_version']}</param>  <!-- /niryo_one/hardware_version -->
+				<param name="use_sim">${mp['use_sim']}</param>  <!-- ~fake_communication -->
+				<!-- Niryo One Communication -->
+				<param name="can_enabled">${mp['can_enabled']}</param>  <!-- ~can_enabled -->
+				<param name="dxl_enabled">${mp['dxl_enabled']}</param>  <!-- ~dxl_enabled -->
+				<param name="niryo_one_hw_check_connection_frequency">${mp['niryo_one_hw_check_connection_frequency']}</param>  <!-- niryo_one_hw_check_connection_frequency -->
+				<param name="reboot">${mp['reboot']}</param>  <!-- /niryo_one/reboot_when_auto_change_version -->
+				<!-- Dxl Communication -->
+				<param name="dxl_uart_device_name">${mp['device_name']}</param>
+				<param name="dxl_baudrate">${mp['uart_baudrate']}</param>
+				<param name="dxl_hardware_control_loop_frequency">${mp['dxl_hw_control_loop_frequency']}</param>
+				<param name="dxl_hw_write_frequency">${mp['dxl_hw_write_frequency']}</param>
+				<param name="dxl_hw_data_read_frequency">${mp['dxl_hw_data_read_frequency']}</param>
+				<param name="dxl_hw_status_read_frequency">${mp['dxl_hw_status_read_frequency']}</param>
+			</hardware>
+			<joint name="joint_4">
+				<param name="id">2</param>
+				<param name="name">Servo Axis 4</param>
+				<param name="type">2</param>  <!-- XL430 -->
+				<command_interface name="position">
+					<param name="min">${limit_low_forearm_rotation}</param>
+					<param name="max">${limit_up_forearm_rotation}</param>
+				</command_interface>
+				<command_interface name="velocity">
+					<param name="max">1.0</param>
+				</command_interface>
+				<command_interface name="torque" />
+				<command_interface name="led" />
+				<state_interface name="position">
+					<param name="initial_value">2047</param>
+				</state_interface>
+				<state_interface name="velocity" />
+				<state_interface name="torque" />
+				<state_interface name="temperature" />
+				<state_interface name="voltage" />
+				<state_interface name="hw_error" />
+				<state_interface name="enabled" />
+			</joint>
+			<joint name="joint_5">
+				<param name="id">3</param>
+				<param name="name">Servo Axis 5</param>
+				<param name="type">2</param>  <!-- XL430 -->
+				<command_interface name="position">
+					<param name="min">${limit_low_wrist_rotation}</param>
+					<param name="max">${limit_up_wrist_rotation}</param>
+				</command_interface>
+				<command_interface name="velocity">
+					<param name="max">1.0</param>
+				</command_interface>
+				<command_interface name="torque" />
+				<command_interface name="led" />
+				<state_interface name="position">
+					<param name="initial_value">2047</param>
+				</state_interface>
+				<state_interface name="velocity" />
+				<state_interface name="torque" />
+				<state_interface name="temperature" />
+				<state_interface name="voltage" />
+				<state_interface name="hw_error" />
+				<state_interface name="enabled" />
+			</joint>
+			<joint name="joint_6">
+				<param name="id">6</param>
+				<param name="name">Servo Axis 6</param>
+				<param name="type">1</param>  <!-- XL320 -->
+				<command_interface name="position">
+					<param name="min">${limit_low_hand_rotation}</param>
+					<param name="max">${limit_up_hand_rotation}</param>
+				</command_interface>
+				<command_interface name="velocity">
+					<param name="max">1.0</param>
+				</command_interface>
+				<command_interface name="torque" />
+				<command_interface name="led" />
+				<state_interface name="position">
+					<param name="initial_value">511</param>
+				</state_interface>
+				<state_interface name="velocity" />
+				<state_interface name="torque" />
+				<state_interface name="temperature" />
+				<state_interface name="voltage" />
+				<state_interface name="hw_error" />
+				<state_interface name="enabled" />
 			</joint>
 		</ros2_control>

File: src/niryo_one_hardware/description/urdf/niryo_one.urdf.xacro (robot description, xacro)
@@ -1,7 +1,30 @@
 <?xml version="1.0"?>
 <robot xmlns:xacro="http://www.ros.org/wiki/xacro" name="niryo_one">
+	<!-- Properties -->
+	<xacro:property name="distance_origin_shoulder_z" value="0.103" scope="global" />
+	<xacro:property name="distance_shoulder_arm_z" value="0.080" scope="global" />
+	<xacro:property name="distance_arm_elbow_x" value="0.210" scope="global" />
+	<xacro:property name="distance_arm_elbow_y" value="0.0" scope="global" />
+	<xacro:property name="distance_elbow_forearm_x" value="0.0415" scope="global" />
+	<xacro:property name="distance_elbow_forearm_y" value="0.030" scope="global" />
+	<xacro:property name="distance_forearm_wrist_z" value="0.180" scope="global" />
+	<xacro:property name="distance_wrist_hand_x" value="0.0164" scope="global" />
+	<xacro:property name="distance_wrist_hand_y" value="-0.0055" scope="global" />
+	<xacro:property name="distance_hand_tool" value="0.0073" scope="global" />
+	<xacro:property name="PI" value="3.14159265359" scope="global" />
+	<xacro:property name="limit_low_shoulder_rotation" value="-3.05433" scope="global" />
+	<xacro:property name="limit_up_shoulder_rotation" value="3.05433" scope="global" />
+	<xacro:property name="limit_low_arm_rotation" value="-1.57080" scope="global" />
+	<xacro:property name="limit_up_arm_rotation" value="0.640187" scope="global" />
+	<xacro:property name="limit_low_elbow_rotation" value="-1.397485" scope="global" />
+	<xacro:property name="limit_up_elbow_rotation" value="${PI/2}" scope="global" />
+	<xacro:property name="limit_low_forearm_rotation" value="-3.05433" scope="global" />
+	<xacro:property name="limit_up_forearm_rotation" value="3.05433" scope="global" />
+	<xacro:property name="limit_low_wrist_rotation" value="-1.74533" scope="global" />
+	<xacro:property name="limit_up_wrist_rotation" value="1.91986" scope="global" />
+	<xacro:property name="limit_low_hand_rotation" value="-2.57436" scope="global" />
+	<xacro:property name="limit_up_hand_rotation" value="2.57436" scope="global" />
 	<!-- Import niryo_one macro -->
-	<!-- <xacro:include filename="$(find niryo_one_description)/urdf/v2/niryo_one.urdf.xacro" /> -->
-	<xacro:include filename="$(find niryo_one_description)/urdf/v2/niryo_one_description.urdf.xacro" />
+	<xacro:include filename="$(find niryo_one_description)/urdf/v2/niryo_one_description.urdf.xacro"/>
 	<xacro:niryo_one_description />
 	<!-- Import niryo_one_ros2_control description -->

Commit message: Moveit_config package

File: src/niryo_one_description/urdf/v2/niryo_one_description.urdf.xacro (robot description, xacro)
@@ -113,4 +113,3 @@
 		</joint>
 	</xacro:macro>
-	<xacro:niryo_one_description/>
 </robot>

File: src/niryo_one_hardware/description/ros2_control/niryo_one.ros2_control.xacro (robot description, xacro)
@@ -4,4 +4,16 @@
 	<xacro:property name="params_path" value="$(arg params_path)" />
 	<xacro:property name="mp" value="${xacro.load_yaml(params_path)}" />
+	<xacro:property name="motor_type_xl320" value="1" />
+	<xacro:property name="motor_type_xl430" value="2" />
+	<xacro:property name="xl320_total_angle" value="296.67" />
+	<xacro:property name="xl320_max_position" value="1022" />
+	<xacro:property name="xl320_min_position" value="0" />
+	<xacro:property name="xl320_middle_position" value="511" />
+	<xacro:property name="xl320_total_range_position" value="1023" />
+	<xacro:property name="xl430_total_angle" value="360.36" />
+	<xacro:property name="xl430_max_position" value="4094" />
+	<xacro:property name="xl430_min_position" value="0" />
+	<xacro:property name="xl430_middle_position" value="2047" />
+	<xacro:property name="xl430_total_range_position" value="4095" />
 	<xacro:macro name="niryo_one_ros2_control" params="name">
 		<ros2_control name="${name}_can" type="system">
@@ -74,7 +86,5 @@
 				<command_interface name="torque" />
 				<command_interface name="mirco_steps" />
-				<command_interface name="max_effort">
-					<param name="max">1</param>
-				</command_interface>
+				<command_interface name="max_effort" />
 				<state_interface name="position">
 					<param name="initial_value">${mp['home_position_1']}</param>
@@ -118,7 +128,5 @@
 				<command_interface name="torque" />
 				<command_interface name="mirco_steps" />
-				<command_interface name="max_effort">
-					<param name="max">1</param>
-				</command_interface>
+				<command_interface name="max_effort" />
 				<state_interface name="position">
 					<param name="initial_value">${mp['home_position_2']}</param>
@@ -162,7 +170,5 @@
 				<command_interface name="torque" />
 				<command_interface name="mirco_steps" />
-				<command_interface name="max_effort">
-					<param name="max">1</param>
-				</command_interface>
+				<command_interface name="max_effort" />
 				<state_interface name="position">
 					<param name="initial_value">${mp['home_position_3']}</param>
@@ -205,9 +211,11 @@
 				<param name="dxl_hw_data_read_frequency">${mp['dxl_hw_data_read_frequency']}</param>
 				<param name="dxl_hw_status_read_frequency">${mp['dxl_hw_status_read_frequency']}</param>
+				<param name="allowed_dxl_ids">${mp['allowed_dxl_ids']}</param>
 			</hardware>
 			<joint name="joint_4">
 				<param name="id">2</param>
 				<param name="name">Servo Axis 4</param>
-				<param name="type">2</param>  <!-- XL430 -->
+				<param name="type">${motor_type_xl430}</param>
+				<param name="home_position">${xl430_middle_position}</param>
 				<command_interface name="position">
 					<param name="min">${limit_low_forearm_rotation}</param>
@@ -221,5 +229,5 @@
 				<command_interface name="led" />
 				<state_interface name="position">
-					<param name="initial_value">2047</param>
+					<param name="initial_value">${xl430_middle_position}</param>
 				</state_interface>
 				<state_interface name="velocity" />
@@ -233,5 +241,6 @@
 				<param name="id">3</param>
 				<param name="name">Servo Axis 5</param>
-				<param name="type">2</param>  <!-- XL430 -->
+				<param name="type">${motor_type_xl430}</param>
+				<param name="home_position">${xl430_middle_position}</param>
 				<command_interface name="position">
 					<param name="min">${limit_low_wrist_rotation}</param>
@@ -245,5 +254,5 @@
 				<command_interface name="led" />
 				<state_interface name="position">
-					<param name="initial_value">2047</param>
+					<param name="initial_value">${xl430_middle_position}</param>
 				</state_interface>
 				<state_interface name="velocity" />
@@ -257,5 +266,6 @@
 				<param name="id">6</param>
 				<param name="name">Servo Axis 6</param>
-				<param name="type">1</param>  <!-- XL320 -->
+				<param name="type">${motor_type_xl320}</param>
+				<param name="home_position">${xl320_middle_position}</param>
 				<command_interface name="position">
 					<param name="min">${limit_low_hand_rotation}</param>
@@ -294,5 +304,5 @@
 				<command_interface name="led" />
 				<state_interface name="position">
-					<param name="initial_value">511</param>
+					<param name="initial_value">${xl320_middle_position}</param>
 				</state_interface>
 				<state_interface name="velocity" />

Commit message: Added tool and some extra utilities to try and fix servo

File: src/niryo_one_description/urdf/v2/niryo_one_description.urdf.xacro (robot description, xacro)
@@ -105,8 +105,10 @@
 			<axis xyz="0 0 1" />
 		</joint>
-		<joint name="hand_tool_joint" type="fixed">
+		<joint name="tool" type="revolute">
 			<parent link="hand_link" />
 			<child link="tool_link" />
 			<origin xyz="0 0 ${distance_hand_tool}" rpy="${-PI/2} ${-PI/2} 0" />
+			<limit effort="1" velocity="1.0" lower="${limit_low_tool_rotation}" upper="${limit_up_tool_rotation}" />
+			<axis xyz="0 0 1" />
 		</joint>
 	</xacro:macro>

File: src/niryo_one_hardware/description/ros2_control/niryo_one.ros2_control.xacro (robot description, xacro)
@@ -288,4 +288,29 @@
 				<state_interface name="enabled" />
 			</joint>
+			<joint name="tool">
+				<param name="id">11</param>
+				<param name="name">Gripper</param>
+				<param name="type">${motor_type_xl320}</param>
+				<param name="home_position">${xl320_middle_position}</param>
+				<command_interface name="position">
+					<param name="min">${limit_low_tool_rotation}</param>
+					<param name="max">${limit_up_tool_rotation}</param>
+					<param name="initial_value">${xl320_middle_position}</param>
+				</command_interface>
+				<command_interface name="velocity">
+					<param name="max">1.0</param>
+				</command_interface>
+				<command_interface name="torque" />
+				<command_interface name="led" />
+				<state_interface name="position">
+					<param name="initial_value">${xl320_middle_position}</param>
+				</state_interface>
+				<state_interface name="velocity" />
+				<state_interface name="torque" />
+				<state_interface name="temperature" />
+				<state_interface name="voltage" />
+				<state_interface name="hw_error" />
+				<state_interface name="enabled" />
+			</joint>
 		</ros2_control>
 	</xacro:macro>

File: src/niryo_one_hardware/description/urdf/niryo_one.urdf.xacro (robot description, xacro)
@@ -25,4 +25,6 @@
 	<xacro:property name="limit_low_hand_rotation" value="-2.57436" scope="global" />
 	<xacro:property name="limit_up_hand_rotation" value="2.57436" scope="global" />
+	<xacro:property name="limit_low_tool_rotation" value="${-PI/2}" scope="global" />
+	<xacro:property name="limit_up_tool_rotation" value="${PI/2}" scope="global" />
 	<!-- Import niryo_one macro -->
 	<xacro:include filename="$(find niryo_one_description)/urdf/v2/niryo_one_description.urdf.xacro"/>
